Commit message: add arm model

File: robot_model/ARM_XML/ARM.urdf (robot description, URDF)
Before this commit: robot ARM, 6 links, 5 joints
Links:
- added link virtual_gripper
Joints:
- added joint virtual_gripper_joint: type revolute, parent Link5, child virtual_gripper, origin xyz=0.4975 0 -0.245 rpy=0 0 0, axis 0 1 0, limit lower=-5000 upper=5000 effort=5000 velocity=5000
