Commit message: update gitignore

File: robot_model/ARM_XML/Xiaotian_Arm_v1.urdf (robot description, URDF)
Before this commit: robot Xiaotian_Arm_v1, 7 links, 6 joints
Links:
- link actuator1: geometry collision mesh filename=./arm_meshes/actuator1.STL; visual mesh filename=./arm_meshes/actuator1.STL
- link actuator2: geometry collision mesh filename=./arm_meshes/actuator2.STL; visual mesh filename=./arm_meshes/actuator2.STL
- link actuator3: geometry collision mesh filename=./arm_meshes/actuator3.STL; visual mesh filename=./arm_meshes/actuator3.STL
- link actuator4: geometry collision mesh filename=./arm_meshes/actuator4.STL; visual mesh filename=./arm_meshes/actuator4.STL
- link actuator5: geometry collision mesh filename=./arm_meshes/actuator5.STL; visual mesh filename=./arm_meshes/actuator5.STL
- link actuator6: geometry collision mesh filename=./arm_meshes/actuator6.STL; visual mesh filename=./arm_meshes/actuator6.STL
- link base_link: geometry collision mesh filename=./arm_meshes/base_link.STL; visual mesh filename=./arm_meshes/base_link.STL
